File: Hardware/ESP32-PoE-ISO_Rev_L.kicad_sch (KiCad schematic)
At the start: 161 parts, among them J1 AudioJack2, Q1 Q12MHz/20pF/10ppm/4P/3.2x2.5mm, Q2 BC817-40(SOT23), Q3 BC817-40(SOT23), T1 LMUN2211LT1G(SOT-23), U1 CH340T(SSOP20W), U10 RT9193-30PB, U2 TPS2376D(SO-8), U3 BL4054B-42TPRN(SOT23-5), U4 LAN8710A-EZC(QFN32)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

Commit message: Cleanup hardware
Parts:
- removed C3: 47uF/6.3V/20%/X5R/C0805, OLIMEX_RLC-FP:C_0805_5MIL_DWS, symbol ESP32-PoE-ISO_Rev_L:C
- removed CONN3, CONN4: STEMMA_I2C_QT, Again:JST_SH4, symbol Again-eagle-import:STEMMA_I2C_QT
- removed D4: 1N5819S4/SOD123, OLIMEX_Diodes-FP:SOD-123_1C-2A_KA, symbol ESP32-PoE-ISO_Rev_L:D_Schottky_Small
- removed L5: FB0805/600R/2A, OLIMEX_RLC-FP:L_0805_5MIL_DWS, symbol ESP32-PoE-ISO_Rev_L:L
- removed MICRO_SD1: TFC-9P-1.7H(ATFFS150A01BR016), OLIMEX_Connectors-FP:uSD(TFC-9P-1.xH(ATFFS150A01BR016)), symbol ESP32-PoE-ISO_Rev_L:MICRO_SD(TFC-9P-1.xH(ATFFS150A01BR016))
- removed R31, R35: 2.2k/R0402, OLIMEX_RLC-FP:R_0402_5MIL_DWS, symbol ESP32-PoE-ISO_Rev_L:R
- removed R36, R37, R39: 10k/R0402, OLIMEX_RLC-FP:R_0402_5MIL_DWS, symbol ESP32-PoE-ISO_Rev_L:R
- removed R40: 10R/R0402, OLIMEX_RLC-FP:R_0402_5MIL_DWS, symbol ESP32-PoE-ISO_Rev_L:R
- removed R46: 220R/R0402, OLIMEX_RLC-FP:R_0402_5MIL_DWS, symbol ESP32-PoE-ISO_Rev_L:R
- removed RM3: RA1206_(4X0603)_4B8_2.2k, OLIMEX_RLC-FP:R_MATRIX_4, symbol ESP32-PoE-ISO_Rev_L:RA1206_(4x0603)_4B8_Smashed
- removed UEXT1: P-B-V-10-LF, OLIMEX_Connectors-FP:GBH-254-SMT-10, symbol ESP32-PoE-ISO_Rev_L:BH10S
Connections:
- net GND: now also C34.2, C35.1, C36.1, U10.5 (IN), U10.7 (OUT), U9.5 (V+)
- net GPIO21/EMAC_TX_EN(RMII): no longer R3.7 (2), RF1.5 (SDA)
- net GPIO22/EMAC_TXD1(RMII): no longer R3.6 (2), RF1.6 (SCL)
- net GPIO32: no longer C33.1, D13.1 (K), R50.1, R53.1
- new net: C33.1, D13.1 (K), R50.1, R53.1
- new net: R3.6 (2), RF1.6 (SCL)
- new net: R3.7 (2), RF1.5 (SDA)
- no-connect marks 20 -> 19
Other:
- note added: "Analog Signal"
- note added: "Current Sensor"
- note added: "Extensions (dev board only)"
- note added: "RFID Tag"
- note removed: "Extensions"
- note removed: "HSPICLK"
- note removed: "HSPID"
- note removed: "HSPIQ"
- note removed: "SD/MMC Card"
- note removed: "STEMMA/I2C Headers"
- note removed: "UEXT"
- company: OLIMEX LTD. -> advin.io
- title: ESP32-PoE-ISO -> ESP32-PoE-ISO - Uplink
- moved on the sheet: ANT1, BUT1, C1, C12, C19, C20, C23, C24, C25, C26, C27, C3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
